File: Analog_Computer_Division_Module/Division_module.kicad_sch (KiCad schematic)
At the start: 33 parts, among them IC1 AD633, U3 DG419BDY-E3, U4 TLE2074IDWR, U5 TLE2074IDWR, U6 DG419BDY-E3

Commit message: cleaned up design and updated README
Parts:
- R10, R14, R15, R9: value 10k -> 100k (0.1p)
- R12, R19, R3, R4, R8: value 100k -> 100k (0.1p)
- R18: value 25k -> 25k (0.1p)
Changed lines of the file:
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@@
 			)
 		)
-		(property "Value" "100k"
+		(property "Value" "100k (0.1p)"
 			(at 142.24 90.17 90)
 			(effects
@@
 			)
 		)
-		(property "Value" "25k"
+		(property "Value" "25k (0.1p)"
 			(at 35.56 124.46 90)
 			(effects
@@
 			)
 		)
-		(property "Value" "10k"
+		(property "Value" "100k (0.1p)"
 			(at 35.56 104.14 90)
 			(effects
@@
 			)
 		)
-		(property "Value" "10k"
+		(property "Value" "100k (0.1p)"
 			(at 35.56 96.52 90)
 			(effects
@@
 			)
 		)
-		(property "Value" "10k"
+		(property "Value" "100k (0.1p)"
 			(at 48.26 107.95 90)
 			(effects
@@
 			)
 		)
-		(property "Value" "100k"
+		(property "Value" "100k (0.1p)"
 			(at 125.73 102.87 90)
 			(effects
@@
 			)
 		)
-		(property "Value" "100k"
+		(property "Value" "100k (0.1p)"
 			(at 35.56 134.62 90)
 			(effects
@@
 			)
 		)
-		(property "Value" "100k"
+		(property "Value" "100k (0.1p)"
 			(at 49.53 22.86 90)
 			(effects
@@
 			)
 		)
-		(property "Value" "100k"
+		(property "Value" "100k (0.1p)"
 			(at 33.02 36.83 90)
 			(effects
@@
 			)
 		)
-		(property "Value" "10k"
+		(property "Value" "100k (0.1p)"
 			(at 43.18 107.95 90)
 			(effects
