File: Analog_Computer_Division_Module/Division_module_Mult.kicad_sch (KiCad schematic)
At the start: 33 parts, among them IC2 AD633, U11 DG419BDY-E3, U12 TLE2074IDWR, U13 TLE2074IDWR, U14 DG419BDY-E3

Commit message: cleaned up design and updated README
Parts:
- R39, R40, R44, R48, R55: value 100k -> 100k (0.1p)
- R45, R46, R50, R51: value 10k -> 100k (0.1p)
- R54: value 25k -> 25k (0.1p)
Changed lines of the file:
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@@
 			)
 		)
-		(property "Value" "10k"
+		(property "Value" "100k (0.1p)"
 			(at 35.56 99.06 90)
 			(effects
@@
 			)
 		)
-		(property "Value" "100k"
+		(property "Value" "100k (0.1p)"
 			(at 49.53 25.4 90)
 			(effects
@@
 		(dnp no)
 		(property "Reference" "R50"
-			(at 45.72 110.49 90)
+			(at 38.1 113.03 90)
 			(effects
 				(font
@@
 			)
 		)
-		(property "Value" "10k"
+		(property "Value" "100k (0.1p)"
 			(at 43.18 110.49 90)
 			(effects
@@
 			)
 		)
-		(property "Value" "25k"
+		(property "Value" "25k (0.1p)"
 			(at 35.56 127 90)
 			(effects
@@
 			)
 		)
-		(property "Value" "10k"
+		(property "Value" "100k (0.1p)"
 			(at 48.26 110.49 90)
 			(effects
@@
 			)
 		)
-		(property "Value" "100k"
+		(property "Value" "100k (0.1p)"
 			(at 125.73 105.41 90)
 			(effects
@@
 			)
 		)
-		(property "Value" "100k"
+		(property "Value" "100k (0.1p)"
 			(at 33.02 39.37 90)
 			(effects
@@
 			)
 		)
-		(property "Value" "100k"
+		(property "Value" "100k (0.1p)"
 			(at 35.56 137.16 90)
 			(effects
@@
 			)
 		)
-		(property "Value" "100k"
+		(property "Value" "100k (0.1p)"
 			(at 142.24 92.71 90)
 			(effects
@@
 			)
 		)
-		(property "Value" "10k"
+		(property "Value" "100k (0.1p)"
 			(at 35.56 106.68 90)
 			(effects
