File: Analog_Computer_Division_Module/power.kicad_sch (KiCad schematic)
At the start: 11 parts, among them J3 Conn_02x05_Odd_Even, Q1 PMV250EPEA, Q2 PMV450ENEA, U1 VCAN16A2, U2 VCAN16A2

Commit message: cleaned up design and updated README
Parts:
- renumbered J3 to J2
Changed lines of the file:
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@@
 		(on_board yes)
 		(dnp no)
-		(property "Reference" "J3"
+		(property "Reference" "J2"
 			(at 45.72 69.85 0)
 			(effects
@@
 			(project "Analog_Computer_Division_Module"
 				(path "/0a59a61b-9959-4bec-abb4-660a54f0221a/26c40e8a-deac-4fc8-906c-0c0758aeae95"
-					(reference "J3")
+					(reference "J2")
 					(unit 1)
 				)
