File: Middleplate/Analog_Computer_Division_Middleplate.kicad_pcb (KiCad board)
At the start: 2 copper layers, 56.6 x 108.5 mm, 18 parts, among them J1 Conn_01x14_Socket

Commit message: cleaned up design and updated README
Parts:
- U1, U2, U3: value ~ -> VCAN16A2-03S-E3-08
