File: Middleplate/Analog_Computer_Division_Middleplate.kicad_sch (KiCad schematic)
At the start: 19 parts, among them J1 Conn_01x14_Socket

Commit message: cleaned up design and updated README
Parts:
- U1, U2, U3: value ~ -> VCAN16A2-03S-E3-08
Changed lines of the file:
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@@
 			)
 		)
-		(property "Value" "~"
+		(property "Value" "VCAN16A2-03S-E3-08"
 			(at 207.01 33.02 0)
 			(effects
@@
 			)
 		)
-		(property "Value" "~"
+		(property "Value" "VCAN16A2-03S-E3-08"
 			(at 224.79 33.02 0)
 			(effects
@@
 			)
 		)
-		(property "Value" "~"
+		(property "Value" "VCAN16A2-03S-E3-08"
 			(at 189.23 33.02 0)
 			(effects
